Commit message: add and test grx config file and agent

File: mani_skill2_real2sim/assets/descriptions/grx_description/GR1T2/urdf/GR1T2_jaw.urdf (robot description, URDF)
Before this commit: robot GR1T2_jaw, 37 links, 36 joints
Links:
- added link left_end_effector_link
- added link right_end_effector_link
Joints:
- added joint left_end_effector_joint: type fixed, parent left_hand_pitch_link, child left_end_effector_link, origin xyz=0 0 -0.135 rpy=0 0 0
- added joint right_end_effector_joint: type fixed, parent right_hand_pitch_link, child right_end_effector_link, origin xyz=0 0 -0.135 rpy=0 0 0
- joint head_pitch_joint: type revolute -> fixed
- joint head_roll_joint: type revolute -> fixed
- joint head_yaw_joint: type revolute -> fixed
- joint left_ankle_pitch_joint: type revolute -> fixed
- joint left_ankle_roll_joint: type revolute -> fixed
- joint left_hip_pitch_joint: type revolute -> fixed
- joint left_hip_roll_joint: type revolute -> fixed
- joint left_hip_yaw_joint: type revolute -> fixed
- joint left_knee_pitch_joint: type revolute -> fixed
- joint right_ankle_pitch_joint: type revolute -> fixed
- joint right_ankle_roll_joint: type revolute -> fixed
- joint right_hip_pitch_joint: type revolute -> fixed
- joint right_hip_roll_joint: type revolute -> fixed
- joint right_hip_yaw_joint: type revolute -> fixed
- joint right_knee_pitch_joint: type revolute -> fixed

Commit message: fix bug:Fixing abnormal left arm movement in the GRX robot(collision)

File: mani_skill2_real2sim/assets/descriptions/grx_description/GR1T2/urdf/GR1T2_jaw.urdf (robot description, URDF)
Before this commit: robot GR1T2_jaw, 39 links, 38 joints
Joints:
- joint right_elbow_pitch_joint: type revolute -> fixed
- joint right_jaw_joint: type revolute -> fixed
- joint right_shoulder_pitch_joint: type revolute -> fixed
- joint right_shoulder_roll_joint: type revolute -> fixed
- joint right_shoulder_yaw_joint: type revolute -> fixed
- joint right_wrist_pitch_joint: type revolute -> fixed
- joint right_wrist_roll_joint: type revolute -> fixed
- joint right_wrist_yaw_joint: type revolute -> fixed
- joint waist_pitch_joint: type revolute -> fixed
- joint waist_roll_joint: type revolute -> fixed
- joint waist_yaw_joint: type revolute -> fixed

Commit message: Transfer control from the left hand to the right hand.

File: mani_skill2_real2sim/assets/descriptions/grx_description/GR1T2/urdf/GR1T2_jaw.urdf (robot description, URDF)
Before this commit: robot GR1T2_jaw, 39 links, 38 joints
Joints:
- joint left_elbow_pitch_joint: type revolute -> fixed
- joint left_jaw_joint: type revolute -> fixed
- joint left_shoulder_pitch_joint: type revolute -> fixed
- joint left_shoulder_roll_joint: type revolute -> fixed
- joint left_shoulder_yaw_joint: type revolute -> fixed
- joint left_wrist_pitch_joint: type revolute -> fixed
- joint left_wrist_roll_joint: type revolute -> fixed
- joint left_wrist_yaw_joint: type revolute -> fixed
- joint right_elbow_pitch_joint: type fixed -> revolute
- joint right_jaw_joint: type fixed -> revolute
- joint right_shoulder_pitch_joint: type fixed -> revolute
- joint right_shoulder_roll_joint: type fixed -> revolute
- joint right_shoulder_yaw_joint: type fixed -> revolute
- joint right_wrist_pitch_joint: type fixed -> revolute
- joint right_wrist_roll_joint: type fixed -> revolute
- joint right_wrist_yaw_joint: type fixed -> revolute
