Commit message: add control script of fourer_6dof_hand

File: mani_skill2_real2sim/assets/descriptions/grx_description/GR1T2/urdf/GR1T2_fourier_hand_6dof_no_leg_no_collision.urdf (robot description, URDF)
Before this commit: robot GR1T2_fourier_hand_6dof, 61 links, 60 joints
Links:
- link L_hand_base_link: geometry visual mesh filename=../meshes/fourier_hand_6dof/L_hand_base_link.STL
- link L_index_intermediate_link: geometry visual mesh filename=../meshes/fourier_hand_6dof/L_index_intermediate_link.STL
- link L_index_proximal_link: geometry visual mesh filename=../meshes/fourier_hand_6dof/L_index_proximal_link.STL
- link L_middle_intermediate_link: geometry visual mesh filename=../meshes/fourier_hand_6dof/L_middle_intermediate_link.STL
- link L_middle_proximal_link: geometry visual mesh filename=../meshes/fourier_hand_6dof/L_middle_proximal_link.STL
- link L_pinky_intermediate_link: geometry visual mesh filename=../meshes/fourier_hand_6dof/L_pinky_intermediate_link.STL
- link L_pinky_proximal_link: geometry visual mesh filename=../meshes/fourier_hand_6dof/L_pinky_proximal_link.STL
- link L_ring_intermediate_link: geometry visual mesh filename=../meshes/fourier_hand_6dof/L_ring_intermediate_link.STL
- link L_ring_proximal_link: geometry visual mesh filename=../meshes/fourier_hand_6dof/L_ring_proximal_link.STL
- link L_thumb_distal_link: geometry visual mesh filename=../meshes/fourier_hand_6dof/L_thumb_distal_link.STL
- link L_thumb_proximal_base_link: geometry visual mesh filename=../meshes/fourier_hand_6dof/L_thumb_proximal_base_link.STL
- link L_thumb_proximal_link: geometry visual mesh filename=../meshes/fourier_hand_6dof/L_thumb_proximal_link.STL
- link R_hand_base_link: geometry visual mesh filename=../meshes/fourier_hand_6dof/R_hand_base_link.STL
- link R_index_intermediate_link: geometry visual mesh filename=../meshes/fourier_hand_6dof/R_index_intermediate_link.STL
- link R_index_proximal_link: geometry visual mesh filename=../meshes/fourier_hand_6dof/R_index_proximal_link.STL
- link R_middle_intermediate_link: mass 0.11535 -> 0.01535; geometry visual mesh filename=../meshes/fourier_hand_6dof/R_middle_intermediate_link.STL
- link R_middle_proximal_link: geometry visual mesh filename=../meshes/fourier_hand_6dof/R_middle_proximal_link.STL
- link R_pinky_intermediate_link: geometry visual mesh filename=../meshes/fourier_hand_6dof/R_pinky_intermediate_link.STL
- link R_pinky_proximal_link: geometry visual mesh filename=../meshes/fourier_hand_6dof/R_pinky_proximal_link.STL
- link R_ring_proximal_link: mass 0.11911771 -> 0.01911771
- link R_thumb_distal_link: geometry visual mesh filename=../meshes/fourier_hand_6dof/R_thumb_distal_link.STL
- link R_thumb_proximal_base_link: geometry visual mesh filename=../meshes/fourier_hand_6dof/R_thumb_proximal_base_link.STL
- link R_thumb_proximal_link: geometry visual mesh filename=../meshes/fourier_hand_6dof/R_thumb_proximal_link.STL
- link base_link: geometry visual mesh filename=../meshes/base_link.STL
- link head_pitch_link: geometry visual mesh filename=../meshes/head_pitch_link.STL
- link head_roll_link: geometry visual mesh filename=../meshes/head_roll_link.STL
- link head_yaw_link: geometry visual mesh filename=../meshes/head_yaw_link.STL
- link imu_link: geometry visual mesh filename=../meshes/imu_link.STL
- link left_hand_pitch_link: geometry visual mesh filename=../meshes/left_hand_pitch_link.STL
- link left_hand_roll_link: geometry visual mesh filename=../meshes/left_hand_roll_link.STL
- link left_hand_yaw_link: geometry visual mesh filename=../meshes/left_hand_yaw_link.STL
- link left_upper_arm_yaw_link: geometry visual mesh filename=../meshes/left_upper_arm_yaw_link.STL
- link right_hand_yaw_link: geometry visual mesh filename=../meshes/right_hand_yaw_link.STL
- link right_upper_arm_yaw_link: geometry visual mesh filename=../meshes/right_upper_arm_yaw_link.STL
- link torso_link: geometry visual mesh filename=../meshes/torso_link.STL
