Commit message: close collision of some joints in urdf

File: mani_skill2_real2sim/assets/descriptions/grx_description/GR1T2/urdf/GR1T2_fourier_hand_6dof_no_leg.urdf (robot description, URDF)
Before this commit: robot GR1T2_fourier_hand_6dof, 61 links, 60 joints
Links:
- link R_index_intermediate_link: geometry collision mesh filename=../meshes/fourier_hand_6dof/R_index_intermediate_link.STL; visual mesh filename=../meshes/fourier_hand_6dof/R_index_intermediate_link.STL
- link R_index_proximal_link: geometry collision mesh filename=../meshes/fourier_hand_6dof/R_index_proximal_link.STL; visual mesh filename=../meshes/fourier_hand_6dof/R_index_proximal_link.STL
- link R_middle_intermediate_link: geometry collision mesh filename=../meshes/fourier_hand_6dof/R_middle_intermediate_link.STL; visual mesh filename=../meshes/fourier_hand_6dof/R_middle_intermediate_link.STL
- link R_middle_proximal_link: geometry collision mesh filename=../meshes/fourier_hand_6dof/R_middle_proximal_link.STL; visual mesh filename=../meshes/fourier_hand_6dof/R_middle_proximal_link.STL
- link R_pinky_intermediate_link: geometry collision mesh filename=../meshes/fourier_hand_6dof/R_pinky_intermediate_link.STL; visual mesh filename=../meshes/fourier_hand_6dof/R_pinky_intermediate_link.STL
- link R_pinky_proximal_link: geometry collision mesh filename=../meshes/fourier_hand_6dof/R_pinky_proximal_link.STL; visual mesh filename=../meshes/fourier_hand_6dof/R_pinky_proximal_link.STL
- link R_ring_intermediate_link: geometry collision mesh filename=../meshes/fourier_hand_6dof/R_ring_intermediate_link.STL; visual mesh filename=../meshes/fourier_hand_6dof/R_ring_intermediate_link.STL
- link R_ring_proximal_link: geometry collision mesh filename=../meshes/fourier_hand_6dof/R_ring_proximal_link.STL; visual mesh filename=../meshes/fourier_hand_6dof/R_ring_proximal_link.STL
- link R_thumb_distal_link: geometry collision mesh filename=../meshes/fourier_hand_6dof/R_thumb_distal_link.STL; visual mesh filename=../meshes/fourier_hand_6dof/R_thumb_distal_link.STL
- link R_thumb_proximal_base_link: geometry collision mesh filename=../meshes/fourier_hand_6dof/R_thumb_proximal_base_link.STL; visual mesh filename=../meshes/fourier_hand_6dof/R_thumb_proximal_base_link.STL
- link R_thumb_proximal_link: geometry collision mesh filename=../meshes/fourier_hand_6dof/R_thumb_proximal_link.STL; visual mesh filename=../meshes/fourier_hand_6dof/R_thumb_proximal_link.STL
- link head_pitch_link: geometry collision mesh filename=../meshes/head_pitch_link.STL; visual mesh filename=../meshes/head_pitch_link.STL
- link head_roll_link: geometry collision mesh filename=../meshes/head_roll_link.STL; visual mesh filename=../meshes/head_roll_link.STL
- link imu_link: geometry collision mesh filename=../meshes/imu_link.STL; visual mesh filename=../meshes/imu_link.STL
- link left_hand_pitch_link: geometry collision mesh filename=../meshes/left_hand_pitch_link.STL; visual mesh filename=../meshes/left_hand_pitch_link.STL
- link left_hand_roll_link: geometry collision mesh filename=../meshes/left_hand_roll_link.STL; visual mesh filename=../meshes/left_hand_roll_link.STL

Commit message: change the color of robot right hand & arm

File: mani_skill2_real2sim/assets/descriptions/grx_description/GR1T2/urdf/GR1T2_fourier_hand_6dof_no_leg.urdf (robot description, URDF)
Before this commit: robot GR1T2_fourier_hand_6dof, 61 links, 60 joints
Links:
- link R_pinky_proximal_link: mass 0.01911771 -> 0.11911771
