Commit message: adaptation for fourier_hand_6dof

File: mani_skill2_real2sim/assets/descriptions/grx_description/GR1T2/GR1T2_fourier_hand_6dof_no_leg.urdf (robot description, URDF)
Before this commit: robot GR1T2_fourier_hand_6dof, 61 links, 60 joints
Links:
- link R_index_intermediate_link: geometry collision mesh filename=../meshes/fourier_hand_6dof/R_index_intermediate_link.STL; visual mesh filename=../meshes/fourier_hand_6dof/R_index_intermediate_link.STL
- link R_index_proximal_link: geometry collision mesh filename=../meshes/fourier_hand_6dof/R_index_proximal_link.STL; visual mesh filename=../meshes/fourier_hand_6dof/R_index_proximal_link.STL
- link R_middle_intermediate_link: geometry collision mesh filename=../meshes/fourier_hand_6dof/R_middle_intermediate_link.STL; visual mesh filename=../meshes/fourier_hand_6dof/R_middle_intermediate_link.STL
- link R_middle_proximal_link: geometry collision mesh filename=../meshes/fourier_hand_6dof/R_middle_proximal_link.STL; visual mesh filename=../meshes/fourier_hand_6dof/R_middle_proximal_link.STL
- link R_pinky_intermediate_link: geometry collision mesh filename=../meshes/fourier_hand_6dof/R_pinky_intermediate_link.STL; visual mesh filename=../meshes/fourier_hand_6dof/R_pinky_intermediate_link.STL
- link R_pinky_proximal_link: geometry collision mesh filename=../meshes/fourier_hand_6dof/R_pinky_proximal_link.STL; visual mesh filename=../meshes/fourier_hand_6dof/R_pinky_proximal_link.STL
- link R_ring_intermediate_link: geometry collision mesh filename=../meshes/fourier_hand_6dof/R_ring_intermediate_link.STL; visual mesh filename=../meshes/fourier_hand_6dof/R_ring_intermediate_link.STL
- link R_ring_proximal_link: geometry collision mesh filename=../meshes/fourier_hand_6dof/R_ring_proximal_link.STL; visual mesh filename=../meshes/fourier_hand_6dof/R_ring_proximal_link.STL
- link R_thumb_distal_link: geometry collision mesh filename=../meshes/fourier_hand_6dof/R_thumb_distal_link.STL; visual mesh filename=../meshes/fourier_hand_6dof/R_thumb_distal_link.STL
- link R_thumb_proximal_base_link: geometry collision mesh filename=../meshes/fourier_hand_6dof/R_thumb_proximal_base_link.STL; visual mesh filename=../meshes/fourier_hand_6dof/R_thumb_proximal_base_link.STL
- link R_thumb_proximal_link: geometry collision mesh filename=../meshes/fourier_hand_6dof/R_thumb_proximal_link.STL; visual mesh filename=../meshes/fourier_hand_6dof/R_thumb_proximal_link.STL
Joints:
- joint R_index_intermediate_joint: limit lower=-1.74 upper=0 effort=10 velocity=0.8 -> lower=-1.74 upper=0 effort=0 velocity=0; mimic (none) -> joint=R_index_proximal_joint multiplier=1.128 offset=0
- joint R_middle_intermediate_joint: limit lower=-1.74 upper=0 effort=10 velocity=0.8 -> lower=-1.74 upper=0 effort=0 velocity=0; mimic (none) -> joint=R_middle_proximal_joint multiplier=1.131 offset=0
- joint R_pinky_intermediate_joint: limit lower=-1.74 upper=0 effort=10 velocity=0.8 -> lower=-1.74 upper=0 effort=0 velocity=0; mimic (none) -> joint=R_pinky_proximal_joint multiplier=1.129 offset=0
- joint R_ring_intermediate_joint: limit lower=-1.74 upper=0 effort=10 velocity=0.8 -> lower=-1.74 upper=0 effort=0 velocity=0; mimic (none) -> joint=R_ring_proximal_joint multiplier=1.143 offset=0
- joint R_thumb_distal_joint: limit lower=0 upper=1.23 effort=10 velocity=0.8 -> lower=0 upper=1.23 effort=0 velocity=0; mimic (none) -> joint=R_thumb_proximal_pitch_joint multiplier=0.974 offset=0
